File: schematics/TS20_Test_Board/TS20_Test_Board.kicad_pcb (KiCad board)
At the start: 2 copper layers, 114.3 x 59.7 mm, 71 parts, among them J1 Conn_01x06_Pin, SW1 Capacitive Button, SW10 Capacitive Button, SW11 Capacitive Button, SW12 Capacitive Button, SW13 Capacitive Button, SW14 Capacitive Button, SW15 Capacitive Button, SW16 Capacitive Button, SW17 Capacitive Button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

Commit message: add JLC marking
Other:
- board text added: "JLCJLCJLCJLC"
Changed lines of the file:
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@@
+		)
+	)
+	(gr_text "JLCJLCJLCJLC"
+		(at 136.525 58.42 90)
+		(layer "F.SilkS")
+		(effects
+			(font
+				(size 1 1)
+				(thickness 0.225)
+				(bold yes)
+			)
+			(justify left bottom)
 		)
 	)
